File: boards/capactive hub/capactive hub.brd (EAGLE design)
At the start: 96.5 x 59.7 mm, 19 parts

Commit message: updated circuit board designs
Connections:
- net N$15 renamed LEDOUT
Changed lines of the file:
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@@
 <wire x1="76.2" y1="33.02" x2="75.565" y2="33.02" width="0.6096" layer="1"/>
 </signal>
-<signal name="N$15">
+<signal name="LEDOUT">
 <contactref element="CON1" pad="3"/>
 <contactref element="CON2" pad="4"/>
