File: boards/capactive hub/capactive hub.sch (EAGLE design)
At the start: 19 parts

Commit message: updated circuit board designs
Connections:
- net N$15 renamed LEDOUT
Changed lines of the file:
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@@
 <pinref part="CON1" gate="A" pin="5"/>
 <wire x1="111.76" y1="91.44" x2="104.14" y2="91.44" width="0.1524" layer="91"/>
+<label x="104.14" y="91.44" size="1.778" layer="95"/>
 </segment>
 </net>
@@
 <pinref part="CON1" gate="A" pin="4"/>
 <wire x1="111.76" y1="93.98" x2="104.14" y2="93.98" width="0.1524" layer="91"/>
-</segment>
-</net>
-<net name="N$15" class="0">
+<label x="104.14" y="93.98" size="1.778" layer="95"/>
+</segment>
+</net>
+<net name="LEDOUT" class="0">
 <segment>
 <pinref part="CON1" gate="A" pin="3"/>
@@
 <wire x1="111.76" y1="96.52" x2="119.38" y2="96.52" width="0.1524" layer="91"/>
 <wire x1="119.38" y1="96.52" x2="121.92" y2="93.98" width="0.1524" layer="91"/>
-</segment>
-</net>
+<label x="104.14" y="96.52" size="1.778" layer="95"/>
+</segment>
+</net>
