File: boards/compute hub/compute hub.sch (EAGLE design)
At the start: 9 parts, among them J1 JACK2.1MM

Commit message: updated circuit board designs
Connections:
- net LED1: now also ESPLEFT.10; no longer ESPLEFT.13
- net LED2: now also ESPLEFT.11; no longer ESPLEFT.12
- net LED3: now also ESPLEFT.12; no longer ESPLEFT.11
- net LED4: now also ESPLEFT.13; no longer ESPLEFT.10
Other:
- moved on the sheet: CON-HUB1, CON-HUB2, CON-HUB3, CON-HUB4
