File: boards/compute hub - atmega/compute hub.brd (EAGLE design)
At the start: 58.4 x 96.5 mm, 19 parts, among them IC2 ATMEGA88-THIN, J1 JACK2.1MM

Commit message: updated circuits, added test files, fixed images.
Parts:
- moved J1 5.72 mm to (38.7, 75.6)
Connections:
- net GND: now also J1.CONTACT; no longer J1.SHUNT
Routing:
- net +5V: track 144.6 -> 139.8 mm
- net GND: track 192.4 -> 196.7 mm
- net SCK: track 10.8 -> 11.8 mm
Other:
- board size 58.4 x 96.5 mm -> 59.7 x 96.5 mm
