File: boards/compute hub - atmega/compute hub.sch (EAGLE design)
At the start: 19 parts, among them IC2 ATMEGA88-THIN, J1 JACK2.1MM

Commit message: updated circuits, added test files, fixed images.
Connections:
- net GND: now also J1.CONTACT; no longer J1.SHUNT
